File: Pentagon128_InterfaceBoard.kicad_pcb (KiCad board)
At the start: 2 copper layers, 150 x 60 mm, 49 parts, among them J1 DIN41612_02x32_AB, J10 Tape Out, J11 Tape In, J12 Mini-DIN-6, J14 Barrel_Jack_Switch, J15 Conn_01x07, J2 Conn_02x03_Odd_Even ATmega Pr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, J3 Conn_02x08_Odd_Even Ext Keyb, J4 Conn_02x05_Odd_Even Kempston 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, J5 DE9_Plug Kempston Out SMD, J6 DE15_Plug_HighDensity VGA CRT, J7 Conn_01x04 FDD Power, J8 Conn_01x04 Audio In, J9 AudioJack3, Q1 Q_NPN_BCE, Q2 Q_NPN_BCE, Q3 Q_NPN_BCE, Q4 Q_NPN_BCE, U1 MT8816 PLCC44, U2 ATmega168PA-A, U3 74HC245

Commit message: Critical error fixed: connect RP2040-Zero GND and VCC to pins 31/32 instead of 29/28.
Connections:
- RZ1 pad 1: /pico RGB TO VGA/GP0 -> /pico RGB TO VGA/GP1
- RZ1 pad 10: /pico RGB TO VGA/GP9 -> /pico RGB TO VGA/GP10
- RZ1 pad 11: /pico RGB TO VGA/GP10 -> /pico RGB TO VGA/GP11
- RZ1 pad 12: /pico RGB TO VGA/GP11 -> /pico RGB TO VGA/GP12
- RZ1 pad 13: /pico RGB TO VGA/GP12 -> /pico RGB TO VGA/GP13
- RZ1 pad 14: /pico RGB TO VGA/GP13 -> /pico RGB TO VGA/GP14
- RZ1 pad 15: /pico RGB TO VGA/GP14 -> /pico RGB TO VGA/GP15
- RZ1 pad 2: /pico RGB TO VGA/GP1 -> /pico RGB TO VGA/GP2
- RZ1 pad 3: /pico RGB TO VGA/GP2 -> /pico RGB TO VGA/GP3
- RZ1 pad 4: /pico RGB TO VGA/GP3 -> /pico RGB TO VGA/GP4
- RZ1 pad 5: /pico RGB TO VGA/GP4 -> /pico RGB TO VGA/GP5
- RZ1 pad 6: /pico RGB TO VGA/GP5 -> /pico RGB TO VGA/GP6
- RZ1 pad 7: /pico RGB TO VGA/GP6 -> unconnected-(RZ1-GP7-Pad7)
- RZ1 pad 8: unconnected-(RZ1-GP7-Pad8) -> /pico RGB TO VGA/GP8
- RZ1 pad 9: /pico RGB TO VGA/GP8 -> /pico RGB TO VGA/GP9
